File: CAN_Sniffer_V1/5V-Buck.kicad_sch (KiCad schematic)
At the start: 10 parts, among them U5 TPS5430DDAR

Commit message: iteration 2 routing
Parts:
- removed C19: 47u, Capacitor_SMD:C_0805_2012Metric_Pad1.18x1.45mm_HandSolder, symbol bfr_capacitors:CL21A476MQYNNNE
- removed C20: 10n, Capacitor_SMD:C_0402_1005Metric_Pad0.74x0.62mm_HandSolder, symbol bfr_capacitors:CL05B103KB5NNNC
- removed C22: 22u, Capacitor_SMD:C_0603_1608Metric_Pad1.08x0.95mm_HandSolder, symbol bfr_capacitors:CL10A226MQ8NRNC
- removed R11: 3.3k, Resistor_SMD:R_0402_1005Metric_Pad0.72x0.64mm_HandSolder, symbol bfr_resistors:RMCF0402FT3K30
- removed R9: 10k, Resistor_SMD:R_0402_1005Metric_Pad0.72x0.64mm_HandSolder, symbol bfr_resistors:RMCF0402FT10K0
- added C13: 470p, Capacitor_SMD:C_0603_1608Metric_Pad1.08x0.95mm_HandSolder, symbol bfr_capacitors:06035C471J4Z2A
- added C19: 100u, Capacitor_THT:CP_Radial_D8.0mm_P3.50mm, symbol bfr_capacitors:50ZLH100MEFC8X11.5
- added C22: 10n, Capacitor_SMD:C_0805_2012Metric_Pad1.18x1.45mm_HandSolder, symbol bfr_capacitors:08055A103JAT2A
- added R27: 22, Resistor_SMD:R_0402_1005Metric_Pad0.72x0.64mm_HandSolder, symbol bfr_resistors:RMCF0402FT22R0
- added R28: 10k, Resistor_SMD:R_0805_2012Metric_Pad1.20x1.40mm_HandSolder, symbol bfr_resistors:RMCF0805FT10K0
- added R5: 0, Resistor_SMD:R_0805_2012Metric_Pad1.20x1.40mm_HandSolder, symbol bfr_resistors:RMCF0805ZT0R00
- added R9: 3.3k, Resistor_SMD:R_0805_2012Metric_Pad1.20x1.40mm_HandSolder, symbol bfr_resistors:RMCF0805FT3K30
- added TP2: 5V-VSUP, TestPoint:TestPoint_Pad_D1.0mm, symbol Connector:TestPoint
Connections:
- net GND: now also C19.2, R27.1, R9.1
- net at U5.1 (BOOT): now also C22.1
- net at D5.1 (K), L1.1, U5.8 (PH): now also C13.1, C22.2
- net at U5.4 (VSENSE): now also R28.1, R9.2
- net 5V-VSUP: no longer names the net of L1.2
- net 5V-VSUP: now also C19.1, R28.2, R5.1, TP2.1
- net VSUP renamed VSUP_Filtered
- new net: C13.2, R27.2
- new net 5V_VSUP: R5.2
Other:
- note added: "I_in (buck) = (0.6A*3.3V)/(0.95*5V) = 0.417A (assuming efficiency = 95%, I_out = 600mA at 3V3)"
- note added: "LDO max power dissipation (theoretical for onboard): P_D = (150-25)/88 = 1.42W (assuming amb temp = 25 deg C) LDO needed power dissipation: (5-3.3)*0.6 = 1.02W ->should be ok, pls correct if dis estimate is wrong"
- note added: "STM32: 150 mA CAN transceiver: 70 mA LEDs: 30 mA LCD: 45 mA according to datasheet +100mA leakage = 365mA -> using 600mA for buck converter (overestimating to be safe) Calculations: https://docs.google.com/spreadsheets/d/1epLymsTKMYZpcayYR2TrzBTN5FwB9i6HySkqj1IFzzM/edit?usp=sharing"
- note added: "Start with buck converter, if functional then populate"
- note removed: "STM32: 150 mA CAN transceiver: 70 mA LEDs (assume will add some): 120 mA LCD: 3.5+40 mA, assume 150 to be safe (max supply current I_DD plus backlight supply current) +100mA leakage ----------------------------- =590mA ~ 1A (overestimating to be safe) Calculations: https://docs.google.com/spreadsheets/d/1epLymsTKMYZpcayYR2TrzBTN5FwB9i6HySkqj1IFzzM/edit?usp=sharing"
- moved on the sheet: D5, L1
