File: CAN_Sniffer_V1/CAN_transceiver1.kicad_sch (KiCad schematic)
At the start: 5 parts, among them J1 Conn_01x02, U1 MCP2562

Commit message: changed power schematics and STM32, added MicroSD card connector and LCD display
Parts:
- added D1: LED, LED_SMD:LED_0805_2012Metric_Pad1.15x1.40mm_HandSolder, symbol Device:LED
- added Q1: MMBT3906, Package_TO_SOT_SMD:SOT-23, symbol Transistor_BJT:MMBT3906
- added R5: 150, Resistor_SMD:R_0805_2012Metric_Pad1.20x1.40mm_HandSolder, symbol Device:R_US
- added R6: 4.7k, Resistor_SMD:R_0805_2012Metric_Pad1.20x1.40mm_HandSolder, symbol Device:R_US
Connections:
- net GND: now also D1.1 (K)
- net TX: now also R6.2
- new net: D1.2 (A), R5.2
- new net: Q1.1 (B), R6.1
- new net: Q1.3 (C), R5.1
- new net +3.3V: Q1.2 (E)
Other:
- note added: "~30mA forward current, currently is 20mA to be safe (?)"

Commit message: changed power schem, pinouts, first iteration layout
Parts:
- removed C1, C2: 100n, Capacitor_SMD:C_0805_2012Metric_Pad1.18x1.45mm_HandSolder, symbol Device:C
- removed J1: Conn_01x02, Connector_PinSocket_2.54mm:PinSocket_1x02_P2.54mm_Vertical, symbol Connector:Conn_01x02_Socket
- removed R2: 120, Resistor_SMD:R_0805_2012Metric_Pad1.20x1.40mm_HandSolder, symbol Device:R_US
- removed R5: 150, Resistor_SMD:R_0805_2012Metric_Pad1.20x1.40mm_HandSolder, symbol Device:R_US
- removed R6: 4.7k, Resistor_SMD:R_0805_2012Metric_Pad1.20x1.40mm_HandSolder, symbol Device:R_US
- added C1, C5: 100n, Capacitor_SMD:C_0402_1005Metric_Pad0.74x0.62mm_HandSolder, symbol bfr_capacitors:CL05B104KO5NNNC
- added JP1: 2.54mm, Connector_PinHeader_2.54mm:PinHeader_1x03_P2.54mm_Vertical, symbol bfr_connectors:Jumper
- added R2: 4.7k, Resistor_SMD:R_0603_1608Metric_Pad0.98x0.95mm_HandSolder, symbol bfr_resistors:RMCF0603FT4K70
- added R6: 150, Resistor_SMD:R_0603_1608Metric_Pad0.98x0.95mm_HandSolder, symbol bfr_resistors:RMCF0603FT150R
- added R8: 120, Resistor_SMD:R_0402_1005Metric_Pad0.72x0.64mm_HandSolder, symbol bfr_resistors:RMCF0402FT120R
Connections:
- net 3V3: now also C1.1
- net 5V: now also C5.1
- net CANH: now also R8.1
- net CANL: now also JP1.3 (B)
- net GND: now also C1.2, C5.2
- net TX: now also R2.2
- net at D1.2 (A): now also R6.1
- net at Q1.1 (B): now also R2.1
- net at Q1.3 (C): now also R6.2
- new net: JP1.2 (C), R8.2
- no-connect marks 0 -> 1
Other:
- note removed: "~30mA forward current, currently is 20mA to be safe (?)"

Commit message: iteration 2 routing
Parts:
- removed C1, C5: 100n, Capacitor_SMD:C_0402_1005Metric_Pad0.74x0.62mm_HandSolder, symbol bfr_capacitors:CL05B104KO5NNNC
- added C1, C5: 100n, Capacitor_SMD:C_0805_2012Metric_Pad1.18x1.45mm_HandSolder, symbol bfr_capacitors:08051C104KAT4A
- added TP10: TXD, TestPoint:TestPoint_Pad_D1.0mm, symbol Connector:TestPoint
- added TP11: RXD, TestPoint:TestPoint_Pad_D1.0mm, symbol Connector:TestPoint
- added TP5: CANH, TestPoint:TestPoint_Pad_D1.0mm, symbol Connector:TestPoint
- added TP6: CANL, TestPoint:TestPoint_Pad_D1.0mm, symbol Connector:TestPoint
- U1: Digikey PN (none) -> MCP2562FDT-E/SNCT-ND; Digikey link (none) -> https://www.digikey.com/en/products/detail/microchip-techno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
Connections:
- net +3.3V is gone; now on net 3V3: Q1.2 (E)
- net 3V3: now also C1.1
- net 5V: now also C5.1
- net CANH: now also TP5.1
- net CANL: now also TP6.1
- net GND: now also C1.2, C5.2
- net RX: now also TP11.1
- net TX: now also TP10.1
Other:
- moved on the sheet: D1, Q1, R2, R6
