File: CAN_Sniffer_V1/Power.kicad_sch (KiCad schematic)
At the start: 9 parts, among them J1 USB_B_Micro, Q5 SQ2319CES-T1_GE3, U2 AMS1117-3.3

Commit message: iteration 2 routing
Parts:
- removed C16: 10u, Capacitor_SMD:C_0805_2012Metric_Pad1.18x1.45mm_HandSolder, symbol Device:C
- removed C17: 22u, Capacitor_SMD:C_0805_2012Metric_Pad1.18x1.45mm_HandSolder, symbol Device:C
- removed C6: 100n, Capacitor_SMD:C_0402_1005Metric_Pad0.74x0.62mm_HandSolder, symbol bfr_capacitors:CL05B104KB54PNC
- removed D2: TPD2E001DZDR, TPD2E001DZDR:TPD2E001DZDR, symbol TPD2E001DZDR:TPD2E001DZDR
- removed J1: USB_B_Micro, Connector_USB:USB_Micro-AB_Molex_47590-0001, symbol Connector:USB_B_Micro
- removed U2: AMS1117-3.3, Package_TO_SOT_SMD:SOT-223-3_TabPin2, symbol Regulator_Linear:AMS1117-3.3
- added TP1: VSUP-Filtered, TestPoint:TestPoint_Pad_D1.0mm, symbol Connector:TestPoint
- added TP7: GND, TestPoint:TestPoint_Keystone_5015_Micro_Mini, symbol Connector:TestPoint
- Z2: footprint SOD3716X145N -> DDZ13B-7:SOD3716X145N
Connections:
- net GND: now also TP7.1
- net 24V-5V-Buck-Converter/VSUP renamed VSUP_Filtered
- net VSUP_Filtered: now also TP1.1
- no-connect marks 1 -> 0
Other:
- sheet 24V-5V-Buck-Converter ports: added 5V_VSUP, VSUP_Filtered; removed 5V-VSUP, VSUP
- sheet Power-Mux ports: added 5V_VSUP; removed 5V-VSUP
- sheet RJ45-connector ports: added CAN_RX, VSUP_Filtered; removed RX
- note removed: "5V-3.3V LDO"
- note removed: "I_in (buck) = (0.6A*3.3V)/(0.95*5V) = 0.417A (assuming efficiency = 95%, I_out = 600mA at 3V3)"
- note removed: "LDO max power dissipation: P_D = (150-25)/88 = 1.42W (assuming amb temp = 25 deg C) LDO needed power dissipation: (5-3.3)*0.6 = 1.02W ->should be ok, pls correct if dis estimate is wrong"
- note removed: "USB Connector (not onboard)"
- note removed: "Using onboard ST-link USB connector for flashing program only (300mA current limit) Keep jumper JP5 on E5V always, so onboard USB connector never supplies power or sees rest of PCB Changed to unidirectional TVS diodes for ESD protection on USB, USB_ID is floating (device only) RJ45----buck converter----> ---->LDO---->CAN transceiver, LCD, MicroSD card External USB connector---->power mux---->MCU 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"
- moved on the sheet: Q5, R14, Z2

Commit message: sync changes
Parts:
- Z2: Digikey link (none) -> https://www.digikey.com/en/products/detail/diodes-incorpora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
Changed lines of the file:
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@@
+			)
+		)
+		(property "Digikey link" "https://www.digikey.com/en/products/detail/diodes-incorporated/DDZ13B-7/700105"
+			(at 120.65 85.09 90)
+			(effects
+				(font
+					(size 1.27 1.27)
+				)
+				(hide yes)
 			)
 		)
